Commit message: dev, detailed debugging and analysis

File: spinup/examples/pytorch/URDFs/fep/panda.urdf (robot description, URDF)
Before this commit: robot panda, 12 links, 11 joints
Joints:
- joint panda_joint2: type revolute -> fixed

Commit message: changing to 1 dof, failing

File: spinup/examples/pytorch/URDFs/fep/panda.urdf (robot description, URDF)
Before this commit: robot panda, 12 links, 11 joints
Joints:
- joint panda_joint3: type revolute -> fixed
- joint panda_joint4: type revolute -> fixed
- joint panda_joint5: type revolute -> fixed
- joint panda_joint6: type revolute -> fixed
- joint panda_joint7: type revolute -> fixed

Commit message: Fepv0_7

File: spinup/examples/pytorch/URDFs/fep/panda.urdf (robot description, URDF)
Before this commit: robot panda, 12 links, 11 joints
Joints:
- joint panda_joint2: type fixed -> revolute
- joint panda_joint3: type fixed -> revolute
- joint panda_joint4: type fixed -> revolute
- joint panda_joint5: type fixed -> revolute
- joint panda_joint6: type fixed -> revolute
- joint panda_joint7: type fixed -> revolute
