Commit message: modifications added to run on ETH server

File: spinup/examples/pytorch/URDFs/dobot_conveyer.urdf (robot description, URDF)
Before this commit: robot dobot_conveyer, 1 links, 0 joints
Links:
- link base_link: geometry collision mesh filename=/cluster/home/mnobar/code/spinningup/spinup/examples/pytorc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 scale=.020625 .020625 .020625; visual mesh filename=/cluster/home/mnobar/code/spinningup/spinup/examples/pytorc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 scale=.020625 .020625 .020625
