Commit message: Fep_HW_101 resulsts logged

File: spinup/examples/pytorch/URDFs/fep3/panda_corrected_Nosc.urdf (robot description, URDF)
Before this commit: robot panda, 13 links, 12 joints
Links:
- link panda_hand: geometry collision mesh filename=/home/mahdi/catkin_ws/src/franka_ros/franka_description/mes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; visual mesh filename=/home/mahdi/catkin_ws/src/franka_ros/franka_description/mes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
- link panda_leftfinger: geometry collision box size=17.5e-3 15.2e-3 18.5e-3; collision box size=17.5e-3 7e-3 23.5e-3
- link panda_link0: geometry collision mesh filename=/home/mahdi/catkin_ws/src/franka_ros/franka_description/mes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; visual mesh filename=/home/mahdi/catkin_ws/src/franka_ros/franka_description/mes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
- link panda_link1: geometry collision mesh filename=/home/mahdi/catkin_ws/src/franka_ros/franka_description/mes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; visual mesh filename=/home/mahdi/catkin_ws/src/franka_ros/franka_description/mes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
- link panda_link2: geometry collision mesh filename=/home/mahdi/catkin_ws/src/franka_ros/franka_description/mes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; visual mesh filename=/home/mahdi/catkin_ws/src/franka_ros/franka_description/mes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
- link panda_link3: geometry collision mesh filename=/home/mahdi/catkin_ws/src/franka_ros/franka_description/mes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; visual mesh filename=/home/mahdi/catkin_ws/src/franka_ros/franka_description/mes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
- link panda_link4: geometry collision mesh filename=/home/mahdi/catkin_ws/src/franka_ros/franka_description/mes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; visual mesh filename=/home/mahdi/catkin_ws/src/franka_ros/franka_description/mes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
- link panda_link5: geometry collision mesh filename=/home/mahdi/catkin_ws/src/franka_ros/franka_description/mes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; visual mesh filename=/home/mahdi/catkin_ws/src/franka_ros/franka_description/mes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
- link panda_link6: geometry collision mesh filename=/home/mahdi/catkin_ws/src/franka_ros/franka_description/mes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; visual mesh filename=/home/mahdi/catkin_ws/src/franka_ros/franka_description/mes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
- link panda_link7: geometry collision mesh filename=/home/mahdi/catkin_ws/src/franka_ros/franka_description/mes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; visual mesh filename=/home/mahdi/catkin_ws/src/franka_ros/franka_description/mes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
- link panda_rightfinger: geometry collision box size=17.5e-3 15.2e-3 18.5e-3; collision box size=17.5e-3 7e-3 23.5e-3

File: spinup/examples/pytorch/URDFs/fep3/panda_corrected_Nosc_biased_1.urdf (robot description, URDF)
Before this commit: robot panda, 13 links, 12 joints
Links:
- link panda_hand: geometry collision mesh filename=/home/mahdi/catkin_ws/src/franka_ros/franka_description/mes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; visual mesh filename=/home/mahdi/catkin_ws/src/franka_ros/franka_description/mes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
- link panda_leftfinger: geometry collision box size=17.5e-3 15.2e-3 18.5e-3; collision box size=17.5e-3 7e-3 23.5e-3
- link panda_link0: geometry collision mesh filename=/home/mahdi/catkin_ws/src/franka_ros/franka_description/mes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; visual mesh filename=/home/mahdi/catkin_ws/src/franka_ros/franka_description/mes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
- link panda_link1: geometry collision mesh filename=/home/mahdi/catkin_ws/src/franka_ros/franka_description/mes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; visual mesh filename=/home/mahdi/catkin_ws/src/franka_ros/franka_description/mes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
- link panda_link2: geometry collision mesh filename=/home/mahdi/catkin_ws/src/franka_ros/franka_description/mes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; visual mesh filename=/home/mahdi/catkin_ws/src/franka_ros/franka_description/mes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
- link panda_link3: geometry collision mesh filename=/home/mahdi/catkin_ws/src/franka_ros/franka_description/mes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; visual mesh filename=/home/mahdi/catkin_ws/src/franka_ros/franka_description/mes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
- link panda_link4: geometry collision mesh filename=/home/mahdi/catkin_ws/src/franka_ros/franka_description/mes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; visual mesh filename=/home/mahdi/catkin_ws/src/franka_ros/franka_description/mes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
- link panda_link5: geometry collision mesh filename=/home/mahdi/catkin_ws/src/franka_ros/franka_description/mes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; visual mesh filename=/home/mahdi/catkin_ws/src/franka_ros/franka_description/mes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
- link panda_link6: geometry collision mesh filename=/home/mahdi/catkin_ws/src/franka_ros/franka_description/mes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; visual mesh filename=/home/mahdi/catkin_ws/src/franka_ros/franka_description/mes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
- link panda_link7: geometry collision mesh filename=/home/mahdi/catkin_ws/src/franka_ros/franka_description/mes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; visual mesh filename=/home/mahdi/catkin_ws/src/franka_ros/franka_description/mes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
- link panda_rightfinger: geometry collision box size=17.5e-3 15.2e-3 18.5e-3; collision box size=17.5e-3 7e-3 23.5e-3
