Commit message: Fep_HW_304, server

File: spinup/examples/pytorch/URDFs/fep3/panda_corrected_Nosc_backup_19062025.urdf (robot description, URDF)
Before this commit: robot panda, 13 links, 12 joints
Links:
- link panda_hand: geometry collision mesh filename=/home/mahdi/catkin_ws/src/franka_ros/franka_description/mes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; visual mesh filename=/home/mahdi/catkin_ws/src/franka_ros/franka_description/mes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
- link panda_leftfinger: geometry collision box size=17.5e-3 15.2e-3 18.5e-3; collision box size=17.5e-3 7e-3 23.5e-3
- link panda_link0: geometry collision mesh filename=/home/mahdi/catkin_ws/src/franka_ros/franka_description/mes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; visual mesh filename=/home/mahdi/catkin_ws/src/franka_ros/franka_description/mes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
- link panda_link1: geometry collision mesh filename=/home/mahdi/catkin_ws/src/franka_ros/franka_description/mes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; visual mesh filename=/home/mahdi/catkin_ws/src/franka_ros/franka_description/mes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
- link panda_link2: geometry collision mesh filename=/home/mahdi/catkin_ws/src/franka_ros/franka_description/mes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; visual mesh filename=/home/mahdi/catkin_ws/src/franka_ros/franka_description/mes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
- link panda_link3: geometry collision mesh filename=/home/mahdi/catkin_ws/src/franka_ros/franka_description/mes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; visual mesh filename=/home/mahdi/catkin_ws/src/franka_ros/franka_description/mes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
- link panda_link4: geometry collision mesh filename=/home/mahdi/catkin_ws/src/franka_ros/franka_description/mes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; visual mesh filename=/home/mahdi/catkin_ws/src/franka_ros/franka_description/mes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
- link panda_link5: geometry collision mesh filename=/home/mahdi/catkin_ws/src/franka_ros/franka_description/mes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; visual mesh filename=/home/mahdi/catkin_ws/src/franka_ros/franka_description/mes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
- link panda_link6: geometry collision mesh filename=/home/mahdi/catkin_ws/src/franka_ros/franka_description/mes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; visual mesh filename=/home/mahdi/catkin_ws/src/franka_ros/franka_description/mes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
- link panda_link7: geometry collision mesh filename=/home/mahdi/catkin_ws/src/franka_ros/franka_description/mes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; visual mesh filename=/home/mahdi/catkin_ws/src/franka_ros/franka_description/mes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
- link panda_rightfinger: geometry collision box size=17.5e-3 15.2e-3 18.5e-3; collision box size=17.5e-3 7e-3 23.5e-3
Joints:
- joint panda_joint1: axis -0.0349 0 1.01 -> 0 0 1; origin xyz=0 0 0.338 rpy=0.002 0.003 0.003 -> xyz=0 0 0.333 rpy=0 0 0
- joint panda_joint2: axis 0.01 0.01 1.04 -> 0 0 1; origin xyz=0.003 -0.003 0.005 rpy=-1.7307963267948966 0.003 0.003 -> xyz=0 0 0 rpy=-1.5707963267948966 0 0
- joint panda_joint3: axis 0 0.01 0.995 -> 0 0 1; origin xyz=0.002 -0.3195 0.003 rpy=1.7307963267948966 0.003 0 -> xyz=0 -0.316 0 rpy=1.5707963267948966 0 0
- joint panda_joint4: axis 0.03 0 1.03 -> 0 0 1; origin xyz=0.0895 0.003 0.003 rpy=1.7197963267948966 0 0.003 -> xyz=0.0825 0 0 rpy=1.5707963267948966 0 0
- joint panda_joint5: axis 0 0.03 1.02 -> 0 0 1; origin xyz=-0.0862 0.381 0.001 rpy=-1.7157963267948966 0.03 -0.03 -> xyz=-0.0825 0.384 0 rpy=-1.5707963267948966 0 0
- joint panda_joint6: axis 0 0 1.02 -> 0 0 1; origin xyz=0 0 0.003 rpy=1.6697963267948966 0.003 0 -> xyz=0 0 0 rpy=1.5707963267948966 0 0
- joint panda_joint7: origin xyz=0.088 -0.001 -0.001 rpy=1.5707963267948966 0 0 -> xyz=0.088 0 0 rpy=1.5707963267948966 0 0

File: spinup/examples/pytorch/URDFs/fep3/panda_corrected_Nosc_biased_1_backup_19062025.urdf (robot description, URDF)
Before this commit: robot panda, 13 links, 12 joints
Links:
- link panda_hand: geometry collision mesh filename=/home/mahdi/catkin_ws/src/franka_ros/franka_description/mes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; visual mesh filename=/home/mahdi/catkin_ws/src/franka_ros/franka_description/mes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
- link panda_leftfinger: geometry collision box size=17.5e-3 15.2e-3 18.5e-3; collision box size=17.5e-3 7e-3 23.5e-3
- link panda_link0: geometry collision mesh filename=/home/mahdi/catkin_ws/src/franka_ros/franka_description/mes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; visual mesh filename=/home/mahdi/catkin_ws/src/franka_ros/franka_description/mes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
- link panda_link1: geometry collision mesh filename=/home/mahdi/catkin_ws/src/franka_ros/franka_description/mes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; visual mesh filename=/home/mahdi/catkin_ws/src/franka_ros/franka_description/mes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
- link panda_link2: geometry collision mesh filename=/home/mahdi/catkin_ws/src/franka_ros/franka_description/mes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; visual mesh filename=/home/mahdi/catkin_ws/src/franka_ros/franka_description/mes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
- link panda_link3: geometry collision mesh filename=/home/mahdi/catkin_ws/src/franka_ros/franka_description/mes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; visual mesh filename=/home/mahdi/catkin_ws/src/franka_ros/franka_description/mes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
- link panda_link4: geometry collision mesh filename=/home/mahdi/catkin_ws/src/franka_ros/franka_description/mes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; visual mesh filename=/home/mahdi/catkin_ws/src/franka_ros/franka_description/mes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
- link panda_link5: geometry collision mesh filename=/home/mahdi/catkin_ws/src/franka_ros/franka_description/mes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; visual mesh filename=/home/mahdi/catkin_ws/src/franka_ros/franka_description/mes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
- link panda_link6: geometry collision mesh filename=/home/mahdi/catkin_ws/src/franka_ros/franka_description/mes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; visual mesh filename=/home/mahdi/catkin_ws/src/franka_ros/franka_description/mes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
- link panda_link7: geometry collision mesh filename=/home/mahdi/catkin_ws/src/franka_ros/franka_description/mes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; visual mesh filename=/home/mahdi/catkin_ws/src/franka_ros/franka_description/mes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
- link panda_rightfinger: geometry collision box size=17.5e-3 15.2e-3 18.5e-3; collision box size=17.5e-3 7e-3 23.5e-3
Joints:
- joint panda_joint1: axis -0.0349 0 1.01 -> 0 0 1; origin xyz=0 0 0.338 rpy=0.002 0.003 0.003 -> xyz=0 0 0.3332 rpy=0 0 0
- joint panda_joint2: axis 0.01 0.01 1.04 -> 0 0 1; origin xyz=0.003 -0.003 0.005 rpy=-1.7307963267948966 0.003 0.003 -> xyz=0.0005 -0.0005 0.0005 rpy=-1.5707963267948966 0 0
- joint panda_joint3: axis 0 0.01 0.995 -> 0 0 1; origin xyz=0.002 -0.3195 0.003 rpy=1.7307963267948966 0.003 0 -> xyz=0.0005 -0.3165 0.0005 rpy=1.5707963267948966 0 0
- joint panda_joint4: axis 0.03 0 1.03 -> 0 0 1; origin xyz=0.0895 0.003 0.003 rpy=1.7197963267948966 0 0.003 -> xyz=0.0835 0.001 0.001 rpy=1.5707963267948966 0 0
- joint panda_joint5: axis 0 0.03 1.02 -> 0 0 1; origin xyz=-0.0862 0.381 0.001 rpy=-1.7157963267948966 0.03 -0.03 -> xyz=-0.0832 0.3825 0.001 rpy=-1.5707963267948966 0 0
- joint panda_joint6: axis 0 0 1.02 -> 0 0 1; origin xyz=0 0 0.003 rpy=1.6697963267948966 0.003 0 -> xyz=0 0 0.001 rpy=1.5707963267948966 0 0
